File: v1.3/KiCad/Duo2_Direwolf.kicad_pcb (KiCad board)
At the start: 2 copper layers, 132 x 74 mm, 80 parts, among them J1 I/O, J2 ARJM11A3-009-AB-ER2-T, J3 UART1, J4 DB9F, U1 LMC555xN, U2 NanoPi_Duo2, U3 ADS1115-Breakout, U4 ULN2803A, U6 DS18S20

Commit message: Update with as-built changes and errata to v1.2. Changes updated in v1.3 for future production.
Parts:
- R6: value 3.74k -> 3.00k
Connections:
- C9 pad 1: Net-(C9-Pad1) -> Net-(U1-DIS)
- R11 pad 1: Net-(R11-Pad1) -> +3V3
- R11 pad 2: Net-(C9-Pad1) -> Net-(U1-DIS)
- U1 pad 6: Net-(R11-Pad1) -> Net-(U1-DIS)
- U1 pad 7: Net-(R11-Pad1) -> Net-(U1-DIS)
Routing:
- net Net-(U1-DIS): track 0.00 -> 21.0 mm
- net Net-(R11-Pad1): track 5.39 -> 0.00 mm
- net +3V3: track 188.1 -> 193.3 mm
- net Net-(C9-Pad1): track 3.04 -> 0.00 mm
- net GND: vias 291 -> 289
