File: v1.3/KiCad/Duo2_Direwolf.kicad_sch (KiCad schematic)
At the start: 80 parts, among them J1 I/O, J2 ARJM11A3-009-AB-ER2-T, J3 UART1, J4 DB9F, U1 LMC555xN, U2 NanoPi_Duo2, U3 ADS1115-Breakout, U4 ULN2803A, U6 DS18S20

Commit message: Update with as-built changes and errata to v1.2. Changes updated in v1.3 for future production.
Parts:
- R6: value 3.74k -> 3.00k
Connections:
- net +3V3: now also R11.1
- net at U1.6 (THR), U1.7 (DIS): now also C9.1, R11.2; no longer R11.1
Other:
- note added: "AN0 15.6VDC max!"
- moved on the sheet: R11
